Commit message: modifica

File: urdf/robot_assignment_1_camera.xacro (robot description, xacro)
@@ -159,13 +159,11 @@
 	      </material>
 	    </visual>
-	    <inertial>
-	      <mass value="1e-5" />
-	      <origin xyz="0 0 0" rpy="0 0 0"/>
-	      <inertia ixx="1e-6" ixy="0" ixz="0" iyy="1e-6" iyz="0" izz="1e-6" />
-	    </inertial>
+	   <xacro:default_inertial mass="0.02"/>
   </link>
-  <joint name="camera_joint" type="fixed">
+  <joint name="camera_joint" type="continuous">
 	    <axis xyz="0 0 1" />
-	    <origin xyz="0 0 0.17" rpy="0 0 0"/>
+        <origin xyz="0.0 0.0 0.17" rpy="0 0 0"/>
+        <dynamics damping="0.1"/>
+        <limit effort="10000" velocity="100" />
 	    <child link="camera_link"/>
 	    <parent link="support_camera_link"/>
